File: CAN-CTL-LIGHTING-STM32.kicad_sch (KiCad schematic)
At the start: 48 parts, among them J1 H GND L, J2 TERM, J3 USART1, J4 LEDA, J5 PWR IN, J6 LEDB, J7 LEDC, J8 LEDD, U1 STM32G0B1, U2 MCP2562-E-SN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

Commit message: silkscreen updates, swapped ground and H on can connector
Parts:
- added unit 6 of U5
- J1: value H GND L -> G H L
- U4, U5: value 74LS07 -> 74xHC07
Connections:
- net CANH: now also J1.2 (Pin_2); no longer J1.1 (Pin_1)
- net CTLD3: now also U5.13; no longer U5.13
- net GND: now also J1.1 (Pin_1); no longer J1.2 (Pin_2)
- net LEDD3: now also U5.12; no longer U5.12
Changed lines of the file:
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@@
 	(wire
 		(pts
-			(xy 330.2 118.11) (xy 318.77 118.11)
-		)
-		(stroke
-			(width 0)
-			(type default)
-		)
-	)
-	(wire
-		(pts
 			(xy 27.94 73.66) (xy 35.56 73.66)
 		)
@@
 	(wire
 		(pts
-			(xy 318.77 120.65) (xy 321.31 120.65)
+			(xy 318.77 120.65) (xy 330.2 120.65)
 		)
 		(stroke
@@
 	(wire
 		(pts
+			(xy 318.77 118.11) (xy 321.31 118.11)
+		)
+		(stroke
+			(width 0)
+			(type default)
+		)
+	)
+	(wire
+		(pts
 			(xy 82.55 34.29) (xy 82.55 38.1)
 		)
@@
 	(wire
 		(pts
-			(xy 330.2 128.27) (xy 330.2 118.11)
+			(xy 330.2 128.27) (xy 330.2 120.65)
 		)
 		(stroke
@@
 	)
 	(label "CANH"
-		(at 321.31 120.65 0)
+		(at 321.31 118.11 0)
 		(effects
 			(font
@@
 			)
 		)
-		(property "Value" "H GND L"
+		(property "Value" "G H L"
 			(at 313.69 111.76 0)
 			(effects
@@
 			)
 		)
-		(property "Value" "74LS07"
+		(property "Value" "74xHC07"
 			(at 278.13 82.55 0)
 			(effects
@@
 			)
 		)
-		(property "Value" "74LS07"
+		(property "Value" "74xHC07"
 			(at 242.57 92.71 0)
 			(effects
@@
 			)
 		)
-		(property "Value" "74LS07"
+		(property "Value" "74xHC07"
 			(at 242.57 71.12 0)
 			(effects
@@
 			)
 		)
-		(property "Value" "74LS07"
+		(property "Value" "74xHC07"
 			(at 278.13 119.38 0)
 			(effects
@@
 			)
 		)
-		(property "Value" "74LS07"
+		(property "Value" "74xHC07"
 			(at 278.13 130.81 0)
 			(effects
@@
 			)
 		)
-		(property "Value" "74LS07"
+		(property "Value" "74xHC07"
 			(at 278.13 107.95 0)
 			(effects
@@
 			)
 		)
-		(property "Value" "74LS07"
+		(property "Value" "74xHC07"
 			(at 278.13 71.12 0)
 			(effects
@@
 			)
 		)
-		(property "Value" "74LS07"
+		(property "Value" "74xHC07"
 			(at 278.13 92.71 0)
 			(effects
@@
 			)
 		)
-		(property "Value" "74LS07"
+		(property "Value" "74xHC07"
 			(at 242.57 130.81 0)
 			(effects
@@
 			)
 		)
-		(property "Value" "74LS07"
+		(property "Value" "74xHC07"
 			(at 242.57 119.38 0)
 			(effects
@@
 			)
 		)
-		(property "Value" "74LS07"
+		(property "Value" "74xHC07"
 			(at 242.57 107.95 0)
 			(effects
@@
 			)
 		)
-		(property "Value" "74LS07"
+		(property "Value" "74xHC07"
 			(at 40.64 119.3799 0)
 			(effects
@@
 			)
 		)
-		(property "Value" "74LS07"
+		(property "Value" "74xHC07"
 			(at 242.57 82.55 0)
 			(effects
@@
 			)
 		)
-		(property "Value" "74LS07"
+		(property "Value" "74xHC07"
 			(at 71.12 119.3799 0)
 			(effects

Commit message: added crystal osc
Parts:
- added COSC1: 100n, Capacitor_SMD:C_0603_1608Metric_Pad1.08x0.95mm_HandSolder, symbol Device:C_Small
- added Y1: 8MHz, Oscillator:Oscillator_SMD_EuroQuartz_XO32-4Pin_3.2x2.5mm_RotB_HandSoldering, symbol Oscillator:SG-5032CAN
Connections:
- net +3.3V: now also COSC1.1, Y1.1 (~{ST}), Y1.4 (VCC)
- net GND: now also COSC1.2, Y1.2 (GND)
- net OSC: now reaches U1.10 (PF0)
- net OSC: now also Y1.3 (OUT)
